Commit message: check-2

File: src/beginner_tutorials/urdf/rover.urdf.xacro (robot description, xacro)
@@ -2,6 +2,6 @@
 <robot xmlns:xacro="http://www.ros.org/wiki/xacro" name="sample_bot">
 <!-- An example of a simple robot with 4 wheels and a body -->
-<xacro:property name="rear_r" value="rear_wheel_right"/>
-<xacro:property name="rear_l" value="rear_wheel_left"/>
+<!-- <xacro:property name="rear_r" value="rear_wheel_right"/>
+<xacro:property name="rear_l" value="rear_wheel_left"/> -->
 <link name="base_footprint"/>
 <link name="base_link">

Commit message: check-3

File: src/beginner_tutorials/urdf/rover.urdf.xacro (robot description, xacro)
@@ -1,7 +1,4 @@
 <?xml version="1.0"?>
 <robot xmlns:xacro="http://www.ros.org/wiki/xacro" name="sample_bot">
-<!-- An example of a simple robot with 4 wheels and a body -->
-<!-- <xacro:property name="rear_r" value="rear_wheel_right"/>
-<xacro:property name="rear_l" value="rear_wheel_left"/> -->
 <link name="base_footprint"/>
 <link name="base_link">

Commit message: check-4

File: src/beginner_tutorials/urdf/rover.urdf.xacro (robot description, xacro)
@@ -1,4 +1,7 @@
 <?xml version="1.0"?>
 <robot xmlns:xacro="http://www.ros.org/wiki/xacro" name="sample_bot">
+<!-- An example of a simple robot with 4 wheels and a body -->
+<xacro:property name="rear_r" value="rear_wheel_right"/>
+<xacro:property name="rear_l" value="rear_wheel_left"/>
 <link name="base_footprint"/>
 <link name="base_link">
